Commit message: corrected wheel joint axis

File: agv_description/urdf/wheel.urdf.xacro (robot description, xacro)
@@ -71,5 +71,5 @@
       <origin xyz="${translateX * base_x_origin_to_wheel_origin} ${translateY * base_y_origin_to_wheel_origin} ${base_z_origin_to_wheel_origin}"
               rpy="${M_PI/2} ${flipY*M_PI} ${M_PI/2}" />
-      <axis xyz="0 1 0"
+      <axis xyz="1 0 0"
             rpy="0 0 0" />
       <limit effort="100"

Commit message: edited wheel collision tag

File: agv_description/urdf/wheel.urdf.xacro (robot description, xacro)
@@ -48,7 +48,7 @@
       </visual>
       <collision>
-        <origin xyz="0 0 0" rpy="0 0 ${M_PI/2}" />
+        <origin xyz="0 0 0" rpy="0 ${M_PI/2} 0" />
         <geometry>
-          <cylinder length="${wheel_width}"
+          <cylinder length="${wheel_width+.03}"
                     radius="${wheel_radius}" />
         </geometry>
