Commit message: created wheel and bot urdf

File: agv_description/urdf/bot.urdf.xacro (robot description, xacro)
@@ -28,5 +28,5 @@
 <robot name="rambler" xmlns:xacro="http://www.ros.org/wiki/xacro">
   <xacro:property name="M_PI" value="3.1415926535897931" />
-  <xacro:property name="ground_clearance" value="0.05" />
+  <xacro:property name="ground_clearance" value=".06" />
   <!-- Included URDF/XACRO Files -->
   <xacro:include filename="$(find agv_description)/urdf/materials.urdf.xacro" />
@@ -39,7 +39,7 @@
   <xacro:property name="base_mass" value="21" />
   <xacro:property name="scale" value="0.001"/>
-  <xacro:property name="base_x_origin_to_wheel_origin" value="0.0" />
-  <xacro:property name="base_y_origin_to_wheel_origin" value="0.0" />
-  <xacro:property name="base_z_origin_to_wheel_origin" value="0.0" />
+  <xacro:property name="base_x_origin_to_wheel_origin" value="0.163" /> <!-- 203.2/2 + 500/2-->
+  <xacro:property name="base_y_origin_to_wheel_origin" value="0.25" /> <!--(70)/4 + 440/2-->
+  <xacro:property name="base_z_origin_to_wheel_origin" value="0.1" />
   <link name="base_link">
     <inertial>
@@ -54,8 +54,8 @@
         <mesh filename="package://agv_description/meshes/bot.stl" scale="${scale} ${scale} ${scale}" />
       </geometry>
-      <material name="Red" />
+      <material name="White" />
     </visual>
     <collision>
-      <origin xyz="0 0 0.1125"
+      <origin xyz="0 0 0.06"
               rpy="${M_PI/2} 0 ${M_PI/2}"/>
       <geometry>
@@ -72,11 +72,7 @@
     <child link="sensor_anchor_link" />
   </joint>
-  <agv_wheel fr="front" lr="left" parent="base_link"
-                 translateX="0" translateY="1" flipY="0" />
-  <agv_wheel fr="front" lr="right" parent="base_link"
-                 translateX="0" translateY="-1" flipY="1" />
-  <agv_wheel fr="rear" lr="left" parent="base_link"
-                 translateX="-1" translateY="1" flipY="0" />
-  <agv_wheel fr="rear" lr="right" parent="base_link"
-                 translateX="-1" translateY="-1" flipY="1" />
+  <agv_wheel fr="front" lr="left" parent="base_link" translateX="1" translateY="1" flipY="0" />
+  <agv_wheel fr="front" lr="right" parent="base_link" translateX="1" translateY="-1" flipY="1" />
+  <agv_wheel fr="rear" lr="left" parent="base_link" translateX="-1" translateY="1" flipY="0" />
+  <agv_wheel fr="rear" lr="right" parent="base_link" translateX="-1" translateY="-1" flipY="1" />
 </robot>

File: agv_description/urdf/wheel.urdf.xacro (robot description, xacro)
@@ -36,11 +36,10 @@
       <inertial>
         <mass value="${wheel_mass}" />
-        <origin xyz="0 0 0" />
+        <origin xyz="0 0 0" rpy="0 0 0" />
         <inertia ixx="1.00" ixy="0.00" ixz="-0.00"
                  iyy="0.707107" iyz="0.707107" izz="0.707107" />
        </inertial>
       <visual>
-        <origin xyz="0 0 0"
-                rpy="${M_PI/2} ${flipY*M_PI} ${M_PI/2}" />
+        <origin xyz="0 0 0" rpy="0 0 0" />
         <geometry>
           <mesh filename="package://agv_description/meshes/wheel1.stl" scale="${scale} ${scale} ${scale}" />
@@ -49,6 +48,5 @@
       </visual>
       <collision>
-        <origin xyz="0 0 0"
-                rpy="${M_PI/2} ${flipY*M_PI} 0" />
+        <origin xyz="0 0 0" rpy="0 0 0" />
         <geometry>
           <cylinder length="${wheel_width}"
@@ -71,6 +69,6 @@
       <parent link="${parent}" />
       <child link="${fr}_${lr}_wheel" />
-      <origin xyz="0 0 0"
-              rpy="0 0 0" />
+      <origin xyz="${translateX * base_x_origin_to_wheel_origin} ${translateY * base_y_origin_to_wheel_origin} ${base_z_origin_to_wheel_origin}"
+              rpy="${M_PI/2} ${flipY*M_PI} ${M_PI/2}" />
       <axis xyz="0 1 0"
             rpy="0 0 0" />

Commit message: cleaned up wheel xacro

File: agv_description/urdf/bot.urdf.xacro (robot description, xacro)
@@ -32,5 +32,4 @@
   <xacro:include filename="$(find agv_description)/urdf/materials.urdf.xacro" />
   <xacro:include filename="$(find agv_description)/urdf/wheel.urdf.xacro" />
-  <!-- <xacro:include filename="$(find agv_description)/urdf/grizzly.gazebo" /> -->
   <!-- Key Dimensions -->
   <xacro:property name="base_length" value="0.491" />

File: agv_description/urdf/wheel.urdf.xacro (robot description, xacro)
@@ -78,13 +78,4 @@
                         friction="0.0" />
     </joint>
-    <!-- Transmission links the joints and the controller -->
-<!--     <transmission name="joint_${fr}_${lr}_wheel_trans"
-                  type="SimpleTransmission">
-      <actuator name="joint_${fr}_${lr}_wheel_motor" >
-          <mechanicalReduction>1</mechanicalReduction>
-          <motorTorqueConstant>1</motorTorqueConstant>
-      </actuator>
-      <joint name="joint_${fr}_${lr}_wheel" />
-    </transmission> -->
-  </xacro:macro>
+      </xacro:macro>
 </robot>

Commit message: added comments

File: agv_description/urdf/bot.urdf.xacro (robot description, xacro)
@@ -38,6 +38,6 @@
   <xacro:property name="base_mass" value="21" />
   <xacro:property name="scale" value="0.001"/>
-  <xacro:property name="base_x_origin_to_wheel_origin" value="0.163" /> <!-- 203.2/2 + 500/2-->
-  <xacro:property name="base_y_origin_to_wheel_origin" value="0.25" /> <!--(70)/4 + 440/2-->
+  <xacro:property name="base_x_origin_to_wheel_origin" value="0.163" /> <!-- 203.2/2 + 500/2 +/-tolerance -->
+  <xacro:property name="base_y_origin_to_wheel_origin" value="0.25" /> <!--(70)/4 + 440/2 +/-tolerance -->
   <xacro:property name="base_z_origin_to_wheel_origin" value="0.1" />
   <link name="base_link">

Commit message: edited bot collision tag

File: agv_description/urdf/bot.urdf.xacro (robot description, xacro)
@@ -53,11 +53,11 @@
         <mesh filename="package://agv_description/meshes/bot.stl" scale="${scale} ${scale} ${scale}" />
       </geometry>
-      <material name="White" />
+      <material name="DarkGrey" />
     </visual>
     <collision>
-      <origin xyz="0 0 0.06"
-              rpy="${M_PI/2} 0 ${M_PI/2}"/>
+      <origin xyz="0 0 .123"
+              rpy="0 0 0"/>
       <geometry>
-         <box size="${base_width} ${base_height} ${base_length}" />
+         <box size="${base_length} ${base_width} ${base_height}" />
       </geometry>
     </collision>

File: agv_description/urdf/wheel.urdf.xacro (robot description, xacro)
@@ -48,5 +48,5 @@
       </visual>
       <collision>
-        <origin xyz="0 0 0" rpy="0 0 0" />
+        <origin xyz="0 0 0" rpy="0 0 ${M_PI/2}" />
         <geometry>
           <cylinder length="${wheel_width}"

Commit message: created agv_simulation package

File: agv_description/urdf/bot.urdf.xacro (robot description, xacro)
@@ -53,5 +53,5 @@
         <mesh filename="package://agv_description/meshes/bot.stl" scale="${scale} ${scale} ${scale}" />
       </geometry>
-      <material name="DarkGrey" />
+      <material name="Grey" />
     </visual>
     <collision>

File: agv_description/urdf/wheel.urdf.xacro (robot description, xacro)
@@ -45,5 +45,5 @@
           <mesh filename="package://agv_description/meshes/wheel1.stl" scale="${scale} ${scale} ${scale}" />
         </geometry>
-        <material name="Grey" />
+        <material name="White" />
       </visual>
       <collision>
@@ -61,5 +61,5 @@
       <kd value="1.0" />
       <fdir1 value="1 0 0" />
-      <material>Gazebo/Grey</material>
+      <material>Gazebo/White</material>
       <turnGravityOff>false</turnGravityOff>
       <selfCollide>true</selfCollide>

Commit message: modified bot_mass

File: agv_description/urdf/bot.urdf.xacro (robot description, xacro)
@@ -27,27 +27,28 @@
 -->
 <robot name="rambler" xmlns:xacro="http://www.ros.org/wiki/xacro">
-  <xacro:property name="M_PI" value="3.1415926535897931" />
-  <xacro:property name="ground_clearance" value=".06" />
   <!-- Included URDF/XACRO Files -->
   <xacro:include filename="$(find agv_description)/urdf/materials.urdf.xacro" />
   <xacro:include filename="$(find agv_description)/urdf/wheel.urdf.xacro" />
   <!-- Key Dimensions -->
+  <xacro:property name="M_PI" value="3.1415926535897931" />
+  <xacro:property name="ground_clearance" value=".07" />
   <xacro:property name="base_length" value="0.491" />
   <xacro:property name="base_width" value="0.44" />
   <xacro:property name="base_height" value="0.125" />
-  <xacro:property name="base_mass" value="21" />
+  <xacro:property name="base_mass" value="30" />
   <xacro:property name="scale" value="0.001"/>
   <xacro:property name="base_x_origin_to_wheel_origin" value="0.163" /> <!-- 203.2/2 + 500/2 +/-tolerance -->
   <xacro:property name="base_y_origin_to_wheel_origin" value="0.25" /> <!--(70)/4 + 440/2 +/-tolerance -->
   <xacro:property name="base_z_origin_to_wheel_origin" value="0.1" />
+  <link name="root_link" />
   <link name="base_link">
     <inertial>
       <mass value="${base_mass}"/>
-      <origin xyz="-.25 -.22 ${ground_clearance}"/>
-      <inertia ixx= "1.000000" ixy= "0.000000" ixz="0.000003" iyy="1.000000" iyz="0.000000" izz="1.000000"/>
+      <origin xyz="0 0 ${ground_clearance+base_height/2}"/>
+      <inertia ixx= "1.000000" ixy= "-0.000000" ixz="0.000000" iyy="1.000000" iyz="0.000000" izz="1.000000"/>
     </inertial>
     <visual>
-      <origin xyz="-.25 -.22 ${ground_clearance}"
-              rpy="${M_PI/2} 0 ${M_PI/2}"/>
+      <origin xyz="0 0 ${ground_clearance+base_height/2}"
+              rpy="${M_PI/2} 0 0"/>
       <geometry>
         <mesh filename="package://agv_description/meshes/bot.stl" scale="${scale} ${scale} ${scale}" />
@@ -63,5 +64,12 @@
     </collision>
   </link>
-  <!--Add a sensor anchor link that points to the center of the robot top plate-->
+  <joint name="root_joint"
+         type="fixed">
+    <origin xyz="0 0 ${ground_clearance}"
+            rpy="0 0 0"/>
+    <parent link="root_link" />
+    <child link="base_link" />
+  </joint>
+  <!--Add a sensor anchor link that points to the center of the robot top plate
    <link name="sensor_anchor_link"/>
   <joint name="sensor_anchor_joint" type="fixed">
@@ -70,5 +78,5 @@
     <parent link="base_link" />
     <child link="sensor_anchor_link" />
-  </joint>
+  </joint>-->
   <agv_wheel fr="front" lr="left" parent="base_link" translateX="1" translateY="1" flipY="0" />
   <agv_wheel fr="front" lr="right" parent="base_link" translateX="1" translateY="-1" flipY="1" />

File: agv_description/urdf/wheel.urdf.xacro (robot description, xacro)
@@ -73,6 +73,4 @@
       <axis xyz="1 0 0"
             rpy="0 0 0" />
-      <limit effort="100"
-             velocity="100" />
       <joint_properties damping="0.0"
                         friction="0.0" />

Commit message: modified wheel alignment

File: agv_description/urdf/bot.urdf.xacro (robot description, xacro)
@@ -36,5 +36,5 @@
   <xacro:property name="base_width" value="0.44" />
   <xacro:property name="base_height" value="0.125" />
-  <xacro:property name="base_mass" value="30" />
+  <xacro:property name="base_mass" value="40" />
   <xacro:property name="scale" value="0.001"/>
   <xacro:property name="base_x_origin_to_wheel_origin" value="0.163" /> <!-- 203.2/2 + 500/2 +/-tolerance -->
@@ -80,6 +80,6 @@
   </joint>-->
   <agv_wheel fr="front" lr="left" parent="base_link" translateX="1" translateY="1" flipY="0" />
-  <agv_wheel fr="front" lr="right" parent="base_link" translateX="1" translateY="-1" flipY="1" />
+  <agv_wheel fr="front" lr="right" parent="base_link" translateX="1" translateY="-1" flipY="0" />
   <agv_wheel fr="rear" lr="left" parent="base_link" translateX="-1" translateY="1" flipY="0" />
-  <agv_wheel fr="rear" lr="right" parent="base_link" translateX="-1" translateY="-1" flipY="1" />
+  <agv_wheel fr="rear" lr="right" parent="base_link" translateX="-1" translateY="-1" flipY="0" />
 </robot>

Commit message: removed planar odometry plugin

File: agv_description/urdf/bot.urdf.xacro (robot description, xacro)
@@ -36,10 +36,23 @@
   <xacro:property name="base_width" value="0.44" />
   <xacro:property name="base_height" value="0.125" />
-  <xacro:property name="base_mass" value="40" />
+  <xacro:property name="base_mass" value="30" />
   <xacro:property name="scale" value="0.001"/>
   <xacro:property name="base_x_origin_to_wheel_origin" value="0.163" /> <!-- 203.2/2 + 500/2 +/-tolerance -->
   <xacro:property name="base_y_origin_to_wheel_origin" value="0.25" /> <!--(70)/4 + 440/2 +/-tolerance -->
   <xacro:property name="base_z_origin_to_wheel_origin" value="0.1" />
-  <link name="root_link" />
+  <gazebo>
+    <plugin name="grizzly_diff_controller"
+            filename="libgrizzly_gazebo_plugins.so">
+      <alwaysOn>true</alwaysOn>
+      <updateRate>100.0</updateRate>
+      <rearLeftJoint>joint_rear_left_wheel</rearLeftJoint>
+      <rearRightJoint>joint_rear_right_wheel</rearRightJoint>
+      <frontLeftJoint>joint_front_left_wheel</frontLeftJoint>
+      <frontRightJoint>joint_front_right_wheel</frontRightJoint>
+      <wheelSeparation>${base_y_origin_to_wheel_origin*2}</wheelSeparation>
+      <wheelDiameter>${wheel_radius*2.0}</wheelDiameter>
+      <torque>100</torque>
+    </plugin>
+  </gazebo>
   <link name="base_link">
     <inertial>
@@ -64,22 +77,36 @@
     </collision>
   </link>
-  <joint name="root_joint"
-         type="fixed">
-    <origin xyz="0 0 ${ground_clearance}"
-            rpy="0 0 0"/>
-    <parent link="root_link" />
-    <child link="base_link" />
-  </joint>
-  <!--Add a sensor anchor link that points to the center of the robot top plate
-   <link name="sensor_anchor_link"/>
-  <joint name="sensor_anchor_joint" type="fixed">
-    <origin xyz="0 0 0"
+  <!--Add a sensor anchor link that points to the center of the robot top plate-->
+  <link name="back_bottom_sensor_link" />
+  <joint name="back_bottom_sensor_joint" type="fixed">
+    <origin xyz=".210 0 .110"
             rpy="0 0 0" />
     <parent link="base_link" />
-    <child link="sensor_anchor_link" />
-  </joint>-->
-  <agv_wheel fr="front" lr="left" parent="base_link" translateX="1" translateY="1" flipY="0" />
-  <agv_wheel fr="front" lr="right" parent="base_link" translateX="1" translateY="-1" flipY="0" />
-  <agv_wheel fr="rear" lr="left" parent="base_link" translateX="-1" translateY="1" flipY="0" />
-  <agv_wheel fr="rear" lr="right" parent="base_link" translateX="-1" translateY="-1" flipY="0" />
+    <child link="back_bottom_sensor_link" />
+  </joint>
+  <link name="back_top_sensor_link" />
+  <joint name="back_top_sensor_joint" type="fixed">
+    <origin xyz=".210 0 .170"
+            rpy="0 0 0" />
+    <parent link="base_link" />
+    <child link="back_top_sensor_link" />
+  </joint>
+  <link name="front_bottom_sensor_link" />
+  <joint name="front_bottom_sensor_joint" type="fixed">
+    <origin xyz="-.210 0 .110"
+            rpy="0 0 0" />
+    <parent link="base_link" />
+    <child link="front_bottom_sensor_link" />
+  </joint>
+  <link name="front_top_sensor_link" />
+  <joint name="front_top_sensor_joint" type="fixed">
+    <origin xyz="-.210 0 .170"
+            rpy="0 0 0" />
+    <parent link="base_link" />
+    <child link="front_top_sensor_link" />
+  </joint>
+  <agv_wheel fr="front" lr="left" parent="base_link" translateX="-1" translateY="1" flipY="0" />
+  <agv_wheel fr="front" lr="right" parent="base_link" translateX="-1" translateY="-1" flipY="0" />
+  <agv_wheel fr="rear" lr="left" parent="base_link" translateX="1" translateY="1" flipY="0" />
+  <agv_wheel fr="rear" lr="right" parent="base_link" translateX="1" translateY="-1" flipY="0" />
 </robot>

File: agv_description/urdf/materials.urdf.xacro (robot description, xacro)
@@ -36,5 +36,5 @@
   </material>
   <material name="Grey">
-    <color rgba="0.3 0.3 0.3 1.0" />
+    <color rgba="0.3 0.3 0.3 0.8" />
   </material>
   <material name="DarkGrey">

File: grizzly/grizzly_description/urdf/base.urdf.xacro (robot description, xacro)
@@ -151,11 +151,7 @@
            velocity="0.5" />
   </joint>
-  <grizzly_wheel fr="front" lr="left" parent="front_axle_link"
-                 translateX="0" translateY="1" flipY="0" />
-  <grizzly_wheel fr="front" lr="right" parent="front_axle_link"
-                 translateX="0" translateY="-1" flipY="1" />
-  <grizzly_wheel fr="rear" lr="left" parent="chassis_link"
-                 translateX="-1" translateY="1" flipY="0" />
-  <grizzly_wheel fr="rear" lr="right" parent="chassis_link"
-                 translateX="-1" translateY="-1" flipY="1" />
+  <grizzly_wheel fr="front" lr="left" parent="front_axle_link" translateX="0" translateY="1" flipY="0" />
+  <grizzly_wheel fr="front" lr="right" parent="front_axle_link" translateX="0" translateY="-1" flipY="1" />
+  <grizzly_wheel fr="rear" lr="left" parent="chassis_link" translateX="-1" translateY="1" flipY="0" />
+  <grizzly_wheel fr="rear" lr="right" parent="chassis_link" translateX="-1" translateY="-1" flipY="1" />
 </robot>

Commit message: removed odom_calc

File: agv_description/urdf/bot.urdf.xacro (robot description, xacro)
@@ -38,5 +38,5 @@
   <xacro:property name="base_mass" value="30" />
   <xacro:property name="scale" value="0.001"/>
-  <xacro:property name="base_x_origin_to_wheel_origin" value="0.163" /> <!-- 203.2/2 + 500/2 +/-tolerance -->
+  <xacro:property name="base_x_origin_to_wheel_origin" value="0.122" /> <!-- 203.2/2 + 500/2 +/-tolerance -->
   <xacro:property name="base_y_origin_to_wheel_origin" value="0.25" /> <!--(70)/4 + 440/2 +/-tolerance -->
   <xacro:property name="base_z_origin_to_wheel_origin" value="0.1" />
@@ -55,4 +55,8 @@
     </plugin>
   </gazebo>
+  <agv_wheel fr="front" lr="left" parent="base_link" translateX="-1" translateY="1" flipY="0" />
+  <agv_wheel fr="front" lr="right" parent="base_link" translateX="-1" translateY="-1" flipY="0" />
+  <agv_wheel fr="rear" lr="left" parent="base_link" translateX="1" translateY="1" flipY="0" />
+  <agv_wheel fr="rear" lr="right" parent="base_link" translateX="1" translateY="-1" flipY="0" />
   <link name="base_link">
     <inertial>
@@ -70,5 +74,5 @@
     </visual>
     <collision>
-      <origin xyz="0 0 .123"
+      <origin xyz="0 0 ${ground_clearance+base_height/2}"
               rpy="0 0 0"/>
       <geometry>
@@ -78,17 +82,17 @@
   </link>
   <!--Add a sensor anchor link that points to the center of the robot top plate-->
-  <link name="back_bottom_sensor_link" />
-  <joint name="back_bottom_sensor_joint" type="fixed">
+  <link name="rear_bottom_sensor_link" />
+  <joint name="rear_bottom_sensor_joint" type="fixed">
     <origin xyz=".210 0 .110"
             rpy="0 0 0" />
     <parent link="base_link" />
-    <child link="back_bottom_sensor_link" />
+    <child link="rear_bottom_sensor_link" />
   </joint>
-  <link name="back_top_sensor_link" />
-  <joint name="back_top_sensor_joint" type="fixed">
+  <link name="rear_top_sensor_link" />
+  <joint name="rear_top_sensor_joint" type="fixed">
     <origin xyz=".210 0 .170"
             rpy="0 0 0" />
     <parent link="base_link" />
-    <child link="back_top_sensor_link" />
+    <child link="rear_top_sensor_link" />
   </joint>
   <link name="front_bottom_sensor_link" />
@@ -106,7 +110,3 @@
     <child link="front_top_sensor_link" />
   </joint>
-  <agv_wheel fr="front" lr="left" parent="base_link" translateX="-1" translateY="1" flipY="0" />
-  <agv_wheel fr="front" lr="right" parent="base_link" translateX="-1" translateY="-1" flipY="0" />
-  <agv_wheel fr="rear" lr="left" parent="base_link" translateX="1" translateY="1" flipY="0" />
-  <agv_wheel fr="rear" lr="right" parent="base_link" translateX="1" translateY="-1" flipY="0" />
 </robot>

Commit message: added indicator at front

File: agv_description/urdf/bot.urdf.xacro (robot description, xacro)
@@ -81,4 +81,17 @@
     </collision>
   </link>
+  <link name="base_frame">
+  <visual>
+    <geometry>
+      <sphere radius="0.02"/>
+    </geometry>
+    <material name="Red"/>
+  </visual>
+</link>
+<joint name="base_link_base_frame" type="fixed">
+  <origin xyz="${base_length/2} 0 0.3" rpy="0 0 0 "/>
+  <parent link="base_link"/>
+  <child link="base_frame"/>
+</joint>
   <!--Add a sensor anchor link that points to the center of the robot top plate-->
   <link name="rear_bottom_sensor_link" />

Commit message: edited urdf to include imu sensor

File: agv_description/urdf/bot.urdf.xacro (robot description, xacro)
@@ -95,5 +95,5 @@
 </joint>
   <!--Add a sensor anchor link that points to the center of the robot top plate-->
-  <link name="rear_bottom_sensor_link" />
+  <!-- <link name="rear_bottom_sensor_link" />
   <joint name="rear_bottom_sensor_joint" type="fixed">
     <origin xyz=".210 0 .110"
@@ -123,3 +123,11 @@
     <child link="front_top_sensor_link" />
   </joint>
+  <link name="rear_bottom_sensor_link" /> -->
+<link name="imu_sensor_link"/>
+  <joint name="imu_sensor_link" type="fixed">
+    <origin xyz="0 0 0"
+            rpy="0 0 0" />
+    <parent link="base_link" />
+    <child link="imu_sensor_link" />
+  </joint>
 </robot>

Commit message: solved errors in common costmap

File: agv_description/urdf/bot.urdf.xacro (robot description, xacro)
@@ -124,10 +124,10 @@
   </joint>
   <link name="rear_bottom_sensor_link" /> -->
-<link name="imu_sensor_link"/>
+<!-- <link name="imu_sensor_link"/>
   <joint name="imu_sensor_link" type="fixed">
     <origin xyz="0 0 0"
             rpy="0 0 0" />
     <parent link="base_link" />
-    <child link="imu_sensor_link" />
-  </joint>
+    <child link="imu_sensor_link" /> -->
+  <!-- </joint> -->
 </robot>
